File: Design/Smart_Lights_X1.brd (EAGLE design)
At the start: 55 x 55 mm, 35 parts, among them IC1 MP1584EN-LF-Z, J1 POWER_JACK, Q1 IRLR2905TRPBF, U1 ESP-32S

Commit message: Fixed DC Jack connection
Connections:
- net GND: now also J1.GND, J1.GNDBREAK; no longer J1.PWR
- net VCC: now also J1.PWR; no longer J1.GND, J1.GNDBREAK
Routing:
- net VCC: track 96.2 -> 84.2 mm
Changed lines of the file:
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@@
 <drawing>
 <settings>
-<setting alwaysvectorfont="yes"/>
+<setting alwaysvectorfont="no"/>
 <setting verticaltext="up"/>
 </settings>
@@
 <contactref element="C1" pad="2"/>
 <contactref element="D1" pad="A"/>
-<contactref element="J1" pad="PWR"/>
 <via x="13.5" y="15" extent="1-16" drill="0.35"/>
 <via x="14.5" y="15" extent="1-16" drill="0.35"/>
@@
 <contactref element="H4" pad="P$8"/>
 <contactref element="H4" pad="P$9"/>
+<contactref element="J1" pad="GNDBREAK"/>
+<contactref element="J1" pad="GND"/>
 <wire x1="52.31778125" y1="49.997409375" x2="51.63784375" y2="51.63373125" width="0" layer="19" extent="1-1"/>
 <wire x1="51.6415125" y1="48.3595625" x2="50.0051875" y2="47.679625" width="0" layer="19" extent="1-1"/>
@@
 <contactref element="C1" pad="1"/>
 <contactref element="IC1" pad="7"/>
-<contactref element="J1" pad="GNDBREAK"/>
-<contactref element="J1" pad="GND"/>
-<wire x1="32.2" y1="7.8624" x2="30.5" y2="7.8624" width="1.27" layer="16"/>
-<wire x1="30.5" y1="7.8624" x2="27.5" y2="4.8624" width="1.27" layer="16"/>
-<wire x1="27.5" y1="4.8624" x2="23.0546" y2="9.3078" width="1.27" layer="16"/>
-<wire x1="23.0546" y1="9.3078" x2="23.0546" y2="17.0994" width="1.27" layer="16"/>
 <wire x1="23.0546" y1="17.0994" x2="23.0546" y2="48.0546" width="1.27" layer="16"/>
 <wire x1="23.0546" y1="48.0546" x2="24.865" y2="49.865" width="1.27" layer="16"/>
@@
 <wire x1="45.5" y1="10" x2="43.3" y2="7.8" width="0.6096" layer="16"/>
 <wire x1="43.3" y1="7.8" x2="32.2624" y2="7.8" width="0.6096" layer="16"/>
-<wire x1="32.2624" y1="7.8" x2="32.2" y2="7.8624" width="0.6096" layer="16"/>
+<contactref element="J1" pad="PWR"/>
+<wire x1="23.0546" y1="17.0994" x2="27.5" y2="12.654" width="1.27" layer="1"/>
+<wire x1="27.5" y1="12.654" x2="27.5" y2="10.8624" width="1.27" layer="1"/>
+<wire x1="27.5" y1="10.8624" x2="32.2624" y2="7.8" width="0" layer="19" extent="16-16"/>
 </signal>
 <signal name="N$15">

Commit message: C2 & C5 Grounded
Changed lines of the file:
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@@
 <contactref element="J1" pad="GNDBREAK"/>
 <contactref element="J1" pad="GND"/>
+<via x="47.1823" y="41.6571" extent="1-16" drill="0.35"/>
 <wire x1="52.31778125" y1="49.997409375" x2="51.63784375" y2="51.63373125" width="0" layer="19" extent="1-1"/>
 <wire x1="51.6415125" y1="48.3595625" x2="50.0051875" y2="47.679625" width="0" layer="19" extent="1-1"/>
@@
 <wire x1="3.363675" y1="6.6300625" x2="2.68740625" y2="4.99221875" width="0" layer="19" extent="1-1"/>
 <wire x1="3.36734375" y1="3.35589375" x2="2.68740625" y2="4.99221875" width="0" layer="19" extent="1-1"/>
-<wire x1="45.5" y1="41.4" x2="47" y2="35.25" width="0" layer="19" extent="1-1"/>
 </signal>
 <signal name="3.3V">
